Commit message: Draw a GLB link mesh in metres, as glTF defines it
A URDF or SDF mesh that names a GLB with no scale drew 1000 times too
large: the page decodes a GLB into millimetres, and only cadgen's own
primitive GLBs carried the 0.001 back to metres. The urdf skill says a
mesh authored in metres needs no scale, and a glTF file is metres by its
spec, so a user's GLB now carries the same conversion a primitive does.
STL and 3MF stay drawn as the numbers they hold (the page reads no 3MF
unit), converted by the mesh scale, which is what the skills document.

The browser fixture and the snapshot test scaled their metre GLBs by
0.001 to cancel the bug; they now omit the scale and draw at the same
size. The urdf and sdf skills say which formats take a scale.

Co-Authored-By: Claude Opus 5.5 <noreply@anthropic.com>

File: packages/ui/src/renderers/robot/__fixtures__/arm.urdf (robot description, URDF)
Before this commit: robot arm, 8 links, 7 joints
Links:
- link head: geometry visual mesh filename=meshes/head.glb
